File: Hardware/Internal.kicad_pcb (KiCad board)
At the start: 2 copper layers, 127 parts, among them J1 SWD, J10 24V_OUT, J11 24V_OUT, J12 24V_OUT, J13 24V_OUT, J14 24V_OUT, J15 CAN, J16 CAN, J17 CAN, J18 CAN, J19 CAN, J2 CAN, J20 CAN, J21 DR16, J22 2.54, J23 2.54, J24 2.54, J3 USB_C_Receptacle_USB2.0, J4 JLINK_SWD, J5 CAN, J6 24V_IN, J7 24V_OUT, J8 24V_OUT, J9 24V_OUT, Q1 S8050, Q2 AO3400A, Q3 AO3400A, SW1 BTN1, SW2 RST, U1 STM32G431CBUx, U2 SIT1042T/3, U3 STM32F103CBT6, U4 RS3236, U5 RY8411, Y1 8MHz, Y3 8MHz

Commit message: fix pcb bug
Parts:
- added C31: 100nF, Capacitor_SMD:C_0603_1608Metric, F.Cu at (137.2, 63.2)
- moved Q1 103.4 mm to (104.3, 157.4)
- moved R8 103.4 mm to (93.1, 159.0)
- moved R7 103.4 mm to (93.1, 157.0)
- moved C25 100.4 mm to (87.9, 149.5)
- moved R14 100.4 mm to (91.9, 149.5)
- moved D11 90.2 mm to (88.8, 157.7)
- moved R24 89.9 mm to (99.9, 139.5)
- moved R26 89.9 mm to (99.9, 144.5)
- moved R27 89.9 mm to (99.9, 147.0)
- moved R25 89.9 mm to (99.9, 142.0)
- moved U1 89.4 mm to (137.9, 127.3)
- moved C14 84.9 mm to (87.9, 142.0)
- moved C26 82.4 mm to (91.9, 134.5)
- moved R15 82.4 mm to (95.9, 134.5)
- moved R16 82.4 mm to (95.9, 137.0)
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Connections:
- J4 pad 1: JLINK_SWDIO -> F103_SWDIO
- J4 pad 2: JLINK_SWCLK -> F103_SWCLK
- U1 pad 13: unconnected-(U1-PA5-Pad13) -> LED0
- U1 pad 14: unconnected-(U1-PA6-Pad14) -> LED1
- U1 pad 15: unconnected-(U1-PA7-Pad15) -> BTN0
- U1 pad 2: LED0 -> unconnected-(U1-PC13-Pad2)
- U1 pad 38: SCREEN_BG -> unconnected-(U1-PA15-Pad38)
- U3 pad 23: Net-(U3-VSS-Pad23) -> GND
- U3 pad 35: Net-(U3-VSS-Pad23) -> GND
- U3 pad 47: Net-(U3-VSS-Pad23) -> GND
- U3 pad 8: unconnected-(U3-VSSA-Pad8) -> GND

Commit message: update PCB
Parts:
- added D13: LED_BLUE, LED_SMD:LED_0603_1608Metric, F.Cu at (206.8, 103.1)
- added D14: LED_BLUE, LED_SMD:LED_0603_1608Metric, F.Cu at (206.8, 107.6)
- added D15: LED_BLUE, LED_SMD:LED_0603_1608Metric, F.Cu at (206.8, 112.0)
- added D16: LED_BLUE, LED_SMD:LED_0603_1608Metric, F.Cu at (206.8, 117.0)
- added D17: LED_BLUE, LED_SMD:LED_0603_1608Metric, F.Cu at (223.3, 103.0)
- added D18: LED_BLUE, LED_SMD:LED_0603_1608Metric, F.Cu at (223.3, 107.6)
- added D19: LED_BLUE, LED_SMD:LED_0603_1608Metric, F.Cu at (223.3, 112.0)
- added D20: LED_BLUE, LED_SMD:LED_0603_1608Metric, F.Cu at (223.3, 117.0)
- added R43: 1K, Resistor_SMD:R_0603_1608Metric, B.Cu at (193.2, 83.8)
- added R44: 1K, Resistor_SMD:R_0603_1608Metric, B.Cu at (193.2, 86.3)
- added R45: 1K, Resistor_SMD:R_0603_1608Metric, B.Cu at (193.2, 88.8)
- added R46: 1K, Resistor_SMD:R_0603_1608Metric, B.Cu at (193.2, 91.3)
- added R47: 1K, Resistor_SMD:R_0603_1608Metric, B.Cu at (193.2, 93.8)
- added R48: 1K, Resistor_SMD:R_0603_1608Metric, B.Cu at (193.2, 96.3)
- added R49: 1K, Resistor_SMD:R_0603_1608Metric, B.Cu at (189.2, 83.8)
- added R50: 1K, Resistor_SMD:R_0603_1608Metric, B.Cu at (189.2, 86.3)
- added R51: 1K, Resistor_SMD:R_0603_1608Metric, F.Cu at (206.8, 104.6)
- added R52: 1K, Resistor_SMD:R_0603_1608Metric, F.Cu at (206.8, 109.1)
- added R53: 1K, Resistor_SMD:R_0603_1608Metric, F.Cu at (206.8, 113.6)
- added R54: 1K, Resistor_SMD:R_0603_1608Metric, F.Cu at (206.8, 118.5)
- added R55: 1K, Resistor_SMD:R_0603_1608Metric, F.Cu at (223.3, 104.6)
- added R56: 1K, Resistor_SMD:R_0603_1608Metric, F.Cu at (223.3, 109.3)
- added R57: 1K, Resistor_SMD:R_0603_1608Metric, F.Cu at (223.3, 113.6)
- added R58: 1K, Resistor_SMD:R_0603_1608Metric, F.Cu at (223.3, 118.6)
- added TP1: TestPoint, TestPoint:TestPoint_THTPad_2.0x2.0mm_Drill1.0mm, F.Cu at (210.0, 103.8)
- added TP2: TestPoint, TestPoint:TestPoint_THTPad_2.0x2.0mm_Drill1.0mm, F.Cu at (210.0, 108.3)
- added TP3: TestPoint, TestPoint:TestPoint_THTPad_2.0x2.0mm_Drill1.0mm, F.Cu at (210.0, 112.9)
- added TP4: TestPoint, TestPoint:TestPoint_THTPad_2.0x2.0mm_Drill1.0mm, F.Cu at (210.1, 117.8)
- added TP5: TestPoint, TestPoint:TestPoint_THTPad_2.0x2.0mm_Drill1.0mm, F.Cu at (226.5, 103.8)
- added TP6: TestPoint, TestPoint:TestPoint_THTPad_2.0x2.0mm_Drill1.0mm, F.Cu at (226.5, 108.4)
- added TP7: TestPoint, TestPoint:TestPoint_THTPad_2.0x2.0mm_Drill1.0mm, F.Cu at (226.5, 112.8)
- added TP8: TestPoint, TestPoint:TestPoint_THTPad_2.0x2.0mm_Drill1.0mm, F.Cu at (226.5, 117.8)
- added U7: D1X8K-14BL, Display_7Segment:D1X8K, F.Cu at (201.1, 97.8)
Connections:
- U1 pad 13: LED0 -> unconnected-(U1-PA5-Pad13)
- U1 pad 14: LED1 -> unconnected-(U1-PA6-Pad14)
- U1 pad 15: BTN0 -> unconnected-(U1-PA7-Pad15)
Other:
- board outline added: 55.2 x 60.8 mm
- board text added: "PA0"
- board text added: "PA1"
- board text added: "PA2"
- board text added: "PA3"
- board text added: "PA4"
- board text added: "PA5"
- board text added: "PA6"
- board text added: "PA7"
