File: Hardware/Internal.kicad_sch (KiCad schematic)
At the start: 128 parts, among them J1 SWD, J10 24V_OUT, J11 24V_OUT, J12 24V_OUT, J13 24V_OUT, J14 24V_OUT, J15 CAN, J16 CAN, J17 CAN, J18 CAN, J19 CAN, J2 CAN, J20 CAN, J21 DR16, J22 2.54, J23 2.54, J24 2.54, J3 USB_C_Receptacle_USB2.0, J4 JLINK_SWD, J5 CAN, J6 24V_IN, J7 24V_OUT, J8 24V_OUT, J9 24V_OUT, Q1 S8050, Q2 AO3400A, Q3 AO3400A, SW1 BTN1, SW2 RST, U1 STM32G431CBUx, U2 SIT1042T/3, U3 STM32F103CBT6, U4 RS3236, U5 RY8411, Y1 8MHz, Y3 8MHz

Commit message: fix pcb bug
Connections:
- net F103_SWCLK: now also J4.2 (Pin_2)
- net F103_SWDIO: now also J4.1 (Pin_1)
- net GND: now also U3.23 (VSS), U3.35 (VSS), U3.47 (VSS), U3.8 (VSSA)
- net JLINK_SWCLK: no longer J4.2 (Pin_2)
- net JLINK_SWDIO: no longer J4.1 (Pin_1)
- net SCREEN_BG: no longer names the net of U1.38 (PA15)
- no-connect marks 48 -> 49
Changed lines of the file:
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@@
   (junction (at 85.09 46.355) (diameter 0) (color 0 0 0 0)
+  )
+  (junction (at 337.185 106.68) (diameter 0) (color 0 0 0 0)
   )
   (junction (at 243.84 53.975) (diameter 0) (color 0 0 0 0)
@@
   (no_connect (at 354.965 50.8))
   (no_connect (at 354.965 43.18))
+  (no_connect (at 78.105 173.99))
   (no_connect (at 45.085 204.47))
   (no_connect (at 45.085 207.01))
@@
     (stroke (width 0) (type default))
   )
+  (wire (pts (xy 337.185 106.68) (xy 339.725 106.68))
+    (stroke (width 0) (type default))
+  )
   (wire (pts (xy 172.72 137.795) (xy 175.26 137.795))
     (stroke (width 0) (type default))
@@
     )
   )
+  (global_label "F103_SWCLK" (shape input) (at 259.08 80.01 180) (fields_autoplaced)
+    (effects (font (size 1.27 1.27)) (justify right))
+    (property "Intersheetrefs" "${INTERSHEET_REFS}" (at 244.1811 80.01 0)
+      (effects (font (size 1.27 1.27)) (justify right) hide)
+    )
+  )
   (global_label "PB5" (shape input) (at 311.785 137.16 180) (fields_autoplaced)
     (effects (font (size 1.27 1.27)) (justify right))
@@
     )
   )
+  (global_label "F103_SWDIO" (shape input) (at 259.08 77.47 180) (fields_autoplaced)
+    (effects (font (size 1.27 1.27)) (justify right))
+    (property "Intersheetrefs" "${INTERSHEET_REFS}" (at 244.5439 77.47 0)
+      (effects (font (size 1.27 1.27)) (justify right) hide)
+    )
+  )
   (global_label "+24V_IN" (shape input) (at 36.83 85.725 180) (fields_autoplaced)
     (effects (font (size 1.27 1.27)) (justify right))
@@
     )
   )
-  (global_label "JLINK_SWCLK" (shape input) (at 259.08 80.01 180) (fields_autoplaced)
-    (effects (font (size 1.27 1.27)) (justify right))
-    (property "Intersheetrefs" "${INTERSHEET_REFS}" (at 243.6972 80.01 0)
-      (effects (font (size 1.27 1.27)) (justify right) hide)
-    )
-  )
   (global_label "CAN_TX" (shape input) (at 139.7 135.255 180) (fields_autoplaced)
     (effects (font (size 1.27 1.27)) (justify right))
@@
     )
   )
-  (global_label "SCREEN_BG" (shape input) (at 78.105 173.99 0) (fields_autoplaced)
-    (effects (font (size 1.27 1.27)) (justify left))
-    (property "Intersheetrefs" "${INTERSHEET_REFS}" (at 91.9758 173.99 0)
-      (effects (font (size 1.27 1.27)) (justify left) hide)
-    )
-  )
   (global_label "+24V_IN" (shape input) (at 33.655 46.355 180) (fields_autoplaced)
     (effects (font (size 1.27 1.27)) (justify right))
@@
     (property "Intersheetrefs" "${INTERSHEET_REFS}" (at 87.3192 171.45 0)
       (effects (font (size 1.27 1.27)) (justify left) hide)
-    )
-  )
-  (global_label "JLINK_SWDIO" (shape input) (at 259.08 77.47 180) (fields_autoplaced)
-    (effects (font (size 1.27 1.27)) (justify right))
-    (property "Intersheetrefs" "${INTERSHEET_REFS}" (at 244.06 77.47 0)
-      (effects (font (size 1.27 1.27)) (justify right) hide)
     )
   )
@@
         )
       )
+    )
+  )
+  (symbol (lib_id "power:GND") (at 337.185 106.68 0) (unit 1)
+    (in_bom yes) (on_board yes) (dnp no) (fields_autoplaced)
+    (property "Reference" "#PWR0110" (at 337.185 113.03 0)
+      (effects (font (size 1.27 1.27)) hide)
+    )
+    (property "Value" "GND" (at 337.185 111.76 0)
+      (effects (font (size 1.27 1.27)))
+    )
+    (property "Footprint" "" (at 337.185 106.68 0)
+      (effects (font (size 1.27 1.27)) hide)
+    )
+    (property "Datasheet" "" (at 337.185 106.68 0)
+      (effects (font (size 1.27 1.27)) hide)
+    )
+    (pin "1")
+    (instances
+      (project "Internal"
+        (path "/e93f8570-c610-413f-83c6-534474878841"
+          (reference "#PWR0110") (unit 1)
+        )
+      )

Commit message: update PCB
Parts:
- added D13, D14, D15, D16, D17, D18, D19, D20: LED_BLUE, LED_SMD:LED_0603_1608Metric, symbol Device:LED
- added R43, R44, R45, R46, R47, R48, R49, R50, R51, R52, R53, R54, R55, R56, R57, R58: 1K, Resistor_SMD:R_0603_1608Metric, symbol Device:R
- added TP1, TP2, TP3, TP4, TP5, TP6, TP7, TP8: TestPoint, TestPoint:TestPoint_THTPad_2.0x2.0mm_Drill1.0mm, symbol Connector:TestPoint
- added U7: D1X8K-14BL, Display_7Segment:D1X8K, symbol Display_Character:D1X8K-14BL
Connections:
- net BTN0: no longer U1.15 (PA7)
- net GND: now also D13.1 (K), D14.1 (K), D15.1 (K), D16.1 (K), D17.1 (K), D18.1 (K), D19.1 (K), D20.1 (K), U7.3 (CC), U7.8 (CC)
- net LED0: no longer U1.13 (PA5)
- net LED1: no longer U1.14 (PA6)
- new net: D20.2 (A), R58.2
- new net: R48.2, U7.9 (F)
- new net: D19.2 (A), R57.2
- new net: R46.2, U7.2 (D)
- new net: R49.2, U7.10 (G)
- new net: D15.2 (A), R53.2
- new net: R50.2, U7.5 (DP)
- new net: D17.2 (A), R55.2
- new net: D14.2 (A), R52.2
- new net: D13.2 (A), R51.2
- new net: R43.2, U7.7 (A)
- new net: D16.2 (A), R54.2
- new net: R47.2, U7.1 (E)
- new net: R45.2, U7.4 (C)
- new net: R44.2, U7.6 (B)
- new net: D18.2 (A), R56.2
- new net PA0: R43.1, R51.1, TP1.1
- new net PA1: R44.1, R52.1, TP2.1
- new net PA2: R45.1, R53.1, TP3.1
- new net PA3: R46.1, R54.1, TP4.1
- new net PA4: R47.1, R55.1, TP5.1
- new net PA5: R48.1, R56.1, TP6.1
- new net PA6: R49.1, R57.1, TP7.1
- new net PA7: R50.1, R58.1, TP8.1
